Commit message: fix joint name problem

File: rg2_description/urdf/rg2.urdf.xacro (robot description, xacro)
@@ -79,5 +79,5 @@
         <limit velocity="3.14" effort="10.6" lower="${-pi*0.5}" upper="${pi*0.5}" />
         <!-- <limit velocity="3.14" effort="100" lower="-3" upper="3" /> -->
-        <mimic joint="gripper" multiplier="-1"/>
+        <mimic joint="gripper_joint" multiplier="-1"/>
         <dynamics damping="0.1" friction="0.0" />
         <implicitSpringDamper>True</implicitSpringDamper>
@@ -118,5 +118,5 @@
         <limit velocity="3.14" effort="10.6" lower="${-pi*0.5}" upper="${pi*0.5}" />
         <!-- <limit velocity="3.14" effort="100" lower="-3" upper="3" /> -->
-        <mimic joint="gripper" multiplier="1"/>
+        <mimic joint="gripper_joint" multiplier="1"/>
         <dynamics damping="0.1" friction="0.0" />
         <implicitSpringDamper>True</implicitSpringDamper>
@@ -158,5 +158,5 @@
         <limit velocity="3.14" effort="10.6" lower="${-pi*0.5}" upper="${pi*0.5}" />
         <!-- <limit velocity="3.14" effort="100" lower="-3" upper="3" /> -->
-        <mimic joint="gripper" multiplier="-1"/>
+        <mimic joint="gripper_joint" multiplier="-1"/>
         <dynamics damping="0.1" friction="0.0" />
         <implicitSpringDamper>True</implicitSpringDamper>
@@ -197,5 +197,5 @@
         <limit velocity="3.14" effort="10.6" lower="${-pi*0.5}" upper="${pi*0.5}" />
         <!-- <limit velocity="3.14" effort="100" lower="-3" upper="3" /> -->
-        <mimic joint="gripper" multiplier="1"/>
+        <mimic joint="gripper_joint" multiplier="1"/>
         <dynamics damping="0.1" friction="0.0" />
         <implicitSpringDamper>True</implicitSpringDamper>
@@ -236,5 +236,5 @@
         <limit velocity="3.14" effort="10.6" lower="${-pi*0.5}" upper="${pi*0.5}" />
         <!-- <limit velocity="3.14" effort="100" lower="-3" upper="3" /> -->
-        <mimic joint="gripper" multiplier="-1"/>
+        <mimic joint="gripper_joint" multiplier="-1"/>
         <dynamics damping="0.1" friction="0.0" />
         <implicitSpringDamper>True</implicitSpringDamper>
